File: CR01/final v2.brd (EAGLE design)
At the start: 47.9 x 72.4 mm, 40 parts, among them IC1 REG1117, IC2 TLE5205-2G, IC3 78D2T, Q1 IRFL024N\, Q2 IRFL024N\, U1 ATMEGA328P_TQFP, U2 SN74LVC2GU04DBVR

Commit message: Added controller testing program, reworked motor control library, perormed some unsuccessful testing
Connections:
- new net N$26: SV1.5, U1.2
Changed lines of the file:
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@@
 <wire x1="14.1351" y1="61.2775" x2="13.4239" y2="60.5663" width="0.5" layer="1"/>
+</signal>
+<signal name="N$26">
+<contactref element="SV1" pad="5"/>
+<contactref element="U1" pad="2"/>
+<wire x1="33.3375" y1="7.3025" x2="13.1699" y2="38.5125" width="0" layer="19" extent="1-1"/>
 </signal>
 </signals>

Commit message: final
Connections:
- net N$10 renamed RF_CS
